File: mc-screen-breakout/mc-screen-breakout.kicad_sch (KiCad schematic)
At the start: 27 parts, among them J1 USB_C_Receptacle_PowerOnly_6P, J2 FH28-10S-0.5SH_05_, SW1 NANOT160BP, SW2 NANOT160BP, U1 CMM-3424DT-26165-TR, U2 MDBT50Q-1MV2, Y1 32.768kHz

Commit message: Drew custom switch footprint
Parts:
- SW1, SW2: footprint NANOT160BP:SW_NANOT160BP_CNK -> NANOT160BP:Untitled
Connections:
- net SW1: now also U2.25 (P1.08); no longer U2.37 (P0.13)
- net SW2: now also U2.16 (P0.27); no longer U2.36 (P0.14)
Changed lines of the file:
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@@
 	)
 	(no_connect
-		(at 72.39 106.68)
-	)
-	(no_connect
 		(at 31.75 71.12)
 	)
@@
 	)
 	(no_connect
+		(at 72.39 66.04)
+	)
+	(no_connect
 		(at 31.75 53.34)
 	)
@@
 	)
 	(no_connect
-		(at 31.75 111.76)
-	)
-	(no_connect
 		(at 72.39 88.9)
 	)
@@
 	)
 	(no_connect
+		(at 72.39 68.58)
+	)
+	(no_connect
 		(at 31.75 114.3)
 	)
@@
 		)
 	)
-	(global_label "MIC_DATA"
+	(global_label "SW1"
 		(shape input)
-		(at 31.75 60.96 180)
+		(at 31.75 111.76 180)
 		(fields_autoplaced yes)
 		(effects
@@
 		)
 		(property "Intersheetrefs" "${INTERSHEET_REFS}"
-			(at 20.0562 60.96 0)
+			(at 24.8944 111.76 0)
 			(hide yes)
 			(show_name no)
@@
 		)
 	)
-	(global_label "SW1"
+	(global_label "MIC_DATA"
 		(shape input)
-		(at 72.39 66.04 0)
+		(at 31.75 60.96 180)
 		(fields_autoplaced yes)
 		(effects
@@
 				(size 1.27 1.27)
 			)
-			(justify left)
+			(justify right)
 		)
 		(property "Intersheetrefs" "${INTERSHEET_REFS}"
-			(at 79.2456 66.04 0)
+			(at 20.0562 60.96 0)
 			(hide yes)
 			(show_name no)
@@
 					(size 1.27 1.27)
 				)
-				(justify left)
+				(justify right)
 			)
 		)
@@
 	(global_label "SW2"
 		(shape input)
-		(at 72.39 68.58 0)
+		(at 72.39 106.68 0)
 		(fields_autoplaced yes)
 		(effects
@@
 		)
 		(property "Intersheetrefs" "${INTERSHEET_REFS}"
-			(at 79.2456 68.58 0)
+			(at 79.2456 106.68 0)
 			(hide yes)
 			(show_name no)
@@
 			)
 		)
-		(property "Footprint" "NANOT160BP:SW_NANOT160BP_CNK"
+		(property "Footprint" "NANOT160BP:Untitled"
 			(at 80.01 152.4 0)
 			(hide yes)
@@
 			)
 		)
-		(property "Footprint" "NANOT160BP:SW_NANOT160BP_CNK"
+		(property "Footprint" "NANOT160BP:Untitled"
 			(at 80.01 162.56 0)
 			(hide yes)
